File: eagle/lpc134x.brd (EAGLE design)
At the start: 39.5 x 23.7 mm, 34 parts, among them IC2 LT1763CS8-3.3, Q1 12Mhz, SW1 SWITCH_MCTAEF, T1 Si2301DS, X2 USB-SMD-NS

Commit message: Improved schematic and board.
* Replaced 2xLED with RGB LED
* Replaced third ground pint with 121 (thereby exposing SSP0 and SSP1 completely)
* Realigned labels on bottom
* Exposed SWD pads on bottom
Parts:
- removed LED2: (no value), led:CHIPLED_0805
- removed R2, R3: 150R, rcl:R0402
- added PAD1, PAD2, PAD3, PAD4, PAD5: WIREPADSMD1,27-254, wirepad:SMD1,27-2,54
- added R11, R12, R13: 150R, rcl:R0402
- LED1: device led:CHIPLED_0805 -> microbuilder:RGBLED_PLCC4
- moved LED1 3.75 mm to (36.4, 11.9), turned to 180 degrees
- moved C8 0.67 mm to (12.3, 17.6)
- moved R1 0.67 mm to (15.6, 18.9)
- moved R6 0.67 mm to (22.7, 18.1)
- moved RST 0.67 mm to (16.9, 15.6)
- moved U$2 0.67 mm to (23.8, 16.7)
- moved JP4 0.67 mm to (2.28, 22.0)
- moved IC2 0.67 mm to (7.45, 17.8)
- moved JP3 0.67 mm to (7.36, 22.0)
- moved C2 0.67 mm to (15.2, 5.67)
- moved C1 0.67 mm to (15.6, 11.9)
- moved R8 0.67 mm to (11.3, 2.90)
- moved R9 0.67 mm to (8.05, 2.90)
- moved JP2 0.67 mm to (2.28, 1.69)
- moved IC1 0.67 mm to (24.9, 10.1)
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Connections:
- removed net N$18: LED1.A, R2.2
- removed net N$22: LED2.A, R3.1
- new net 013: IC1.34, R12.1
- new net 121: IC1.26, JP1.1
- new net N$1: LED1.1, R11.2
- new net N$2: LED1.4, R12.2
- new net N$3: LED1.3, R13.2
- net +3V3: now also LED1.2; no longer R2.1, R3.2
- net 010: now also PAD3.1
- net 012: now also R11.1; no longer LED2.C
- net 014: now also R13.1; no longer LED1.C
- net 015: now also PAD4.1
- net 09: now also PAD2.1
- net GND: now also PAD5.1; no longer JP1.1
- net RST: now also PAD1.1
Routing:
- net 121: track 0.00 -> 24.7 mm, vias 0 -> 1
- net N$1: track 0.00 -> 5.60 mm
- net RST: track 16.7 -> 21.2 mm
- net 015: track 11.7 -> 16.1 mm
- net 010: track 12.5 -> 16.9 mm
- net 09: track 11.6 -> 15.9 mm
- net 013: track 0.00 -> 3.19 mm
- net N$3: track 0.00 -> 2.63 mm
- net N$2: track 0.00 -> 2.43 mm
- net 01: track 13.8 -> 15.7 mm
- net N$22: track 1.85 -> 0.00 mm
- net +3V3: track 81.9 -> 80.2 mm
- net N$18: track 1.65 -> 0.00 mm
- net 113: track 5.78 -> 5.12 mm
- net GND: vias 24 -> 23
Other:
- board text added: "00"
- board text added: "121"
- board text added: "MISO0"
- board text added: "MISO1"
- board text added: "MOSI0/SWO"
- board text added: "MOSI1"
- board text added: "SCK0/SWCLK"
- board text added: "SCK1"
- board text added: "SWIO"
- board text removed: "MISO"
- board text removed: "MOSI"
- board text removed: "SCK"
- board text removed: "https://github.com/sebseb7/pentarm13uxx"
