File: eagle/lpc134x.sch (EAGLE design)
At the start: 33 parts, among them IC2 LT1763CS8-3.3, Q1 12Mhz, SW1 SWITCH_MCTAEF, T1 Si2301DS, X2 USB-SMD-NS

Commit message: Improved schematic and board.
* Replaced 2xLED with RGB LED
* Replaced third ground pint with 121 (thereby exposing SSP0 and SSP1 completely)
* Realigned labels on bottom
* Exposed SWD pads on bottom
Parts:
- removed LED2: (no value), led:LEDCHIPLED_0805
- removed R2, R3: 150R, rcl:R-EU_R0402
- added PAD1, PAD2, PAD3, PAD4, PAD5: WIREPADSMD1,27-254, wirepad:WIREPADSMD1,27-254
- added R11, R12, R13: 150R, rcl:R-EU_R0402
- LED1: device led:LEDCHIPLED_0805 -> microbuilder:LED_RGB_PLCC4
Connections:
- removed net N$18: LED1.A, R2.2
- removed net N$22: LED2.A, R3.1
- new net 013: IC1.TDO/PIO0_13/AD2/CT32B1_MAT0, R12.1
- new net 121: IC1.PIO1_21/DCD/MISO1, JP1.1
- new net N$1: LED1.RED, R11.2
- new net N$2: LED1.GRN, R12.2
- new net N$3: LED1.BLUE, R13.2
- net +3V3: now also LED1.ANODE; no longer R2.1, R3.2
- net 010: now also PAD3.P
- net 012: now also R11.1; no longer LED2.C
- net 014: now also R13.1; no longer LED1.C
- net 015: now also PAD4.P
- net 09: now also PAD2.P
- net GND: now also PAD5.P; no longer JP1.1
- net RST: now also PAD1.P
Other:
- note added: "JTAG Pads"
- moved on the sheet: JP1, JP2, JP3, JP4, JP6
